File: Arduino/Sensors/GSR/KiCAD/GSR_LM358/GSR_LM358.sch (KiCad schematic (older format))
At the start: 7 parts, among them IC1 LM358, J1 Finger 1, J2 Finger 2

Commit message: GSR sensor circuit (in KiCAD)
Parts:
- C1, C2: value 100nF -> 0.1uF
Connections:
- wire segments 19 -> 21
Changed lines of the file:
@@
 	6400 3700 6400 4350
-Wire Wire Line
-	5800 3050 5800 3300
-Connection ~ 5800 3050
-Wire Wire Line
-	6150 3050 5800 3050
 Wire Wire Line
 	6150 3250 6150 3300
@@
 P 6150 3150
 F 0 "C2" H 6242 3196 50  0000 L CNN
-F 1 "100nF" H 6242 3105 50  0000 L CNN
+F 1 "0.1uF" H 6242 3105 50  0000 L CNN
 F 2 "" H 6150 3150 50  0001 C CNN
 F 3 "~" H 6150 3150 50  0001 C CNN
@@
 	1    0    0    -1
 $EndComp
-Wire Wire Line
-	5800 3000 5800 3050
 $Comp
 L power:Earth #PWR?
@@
 Wire Wire Line
 	4750 3000 4750 3200
-Wire Wire Line
-	5150 3000 5150 3300
-$Comp
-L power:+5V #PWR?
-U 1 1 63D14ACF
-P 4750 3000
-F 0 "#PWR?" H 4750 2850 50  0001 C CNN
-F 1 "+5V" H 4765 3173 50  0000 C CNN
-F 2 "" H 4750 3000 50  0001 C CNN
-F 3 "" H 4750 3000 50  0001 C CNN
-	1    4750 3000
-	1    0    0    -1
-$EndComp
 Text Notes 7100 3700 0    50   ~ 0
 To Arduino
 Wire Wire Line
 	6400 3700 7050 3700
-$Comp
-L power:+5V #PWR?
-U 1 1 63D12F42
-P 5150 3000
-F 0 "#PWR?" H 5150 2850 50  0001 C CNN
-F 1 "+5V" H 5165 3173 50  0000 C CNN
-F 2 "" H 5150 3000 50  0001 C CNN
-F 3 "" H 5150 3000 50  0001 C CNN
-	1    5150 3000
-	1    0    0    -1
-$EndComp
 Connection ~ 5150 3600
 Wire Wire Line
@@
 P 5150 3400
 F 0 "C1" H 5242 3446 50  0000 L CNN
-F 1 "100nF" H 5242 3355 50  0000 L CNN
+F 1 "0.1uF" H 5242 3355 50  0000 L CNN
 F 2 "" H 5150 3400 50  0001 C CNN
 F 3 "~" H 5150 3400 50  0001 C CNN
@@
 F 3 "ns/lm158.pdf" H 5900 3700 50  0001 C CNN
 	1    5900 3700
-	1    0    0    -1
-$EndComp
-$Comp
-L power:+5V #PWR?
-U 1 1 63D0D48A
-P 5800 3000
-F 0 "#PWR?" H 5800 2850 50  0001 C CNN
-F 1 "+5V" H 5815 3173 50  0000 C CNN
-F 2 "" H 5800 3000 50  0001 C CNN
-F 3 "" H 5800 3000 50  0001 C CNN
-	1    5800 3000
 	1    0    0    -1
 $EndComp
@@
 	0    -1   -1   0
 $EndComp
+Wire Wire Line
+	5150 3000 5150 3300
+Wire Wire Line
+	5150 3000 5800 3000
+Wire Wire Line
+	5150 3000 4750 3000
+Connection ~ 5150 3000
+Wire Wire Line
+	5800 3000 5800 3300
+Connection ~ 5800 3000
+$Comp
+L power:+5V #PWR?
+U 1 1 63D0D48A
+P 5800 3000
+F 0 "#PWR?" H 5800 2850 50  0001 C CNN
+F 1 "+5V" H 5815 3173 50  0000 C CNN
+F 2 "" H 5800 3000 50  0001 C CNN
+F 3 "" H 5800 3000 50  0001 C CNN
+	1    5800 3000
+	1    0    0    -1
+$EndComp
+Wire Wire Line
+	5800 3000 6150 3000
+Wire Wire Line
+	6150 3000 6150 3050
 $EndSCHEMATC
